File: AOTF_Output.kicad_sch (KiCad schematic)
At the start: 0 parts

Commit message: schematic complete
Parts:
- added DSub2: DS1037-25FNAKT74-0CC, Imported:DSUB-TH_DS1037-25FNAKT74-0CC, symbol Imported:DS1037-25FNAKT74-0CC
- added R11, R12, R13, R14, R15, R16, R17, R18: 100k, symbol Device:R
- added R19, R20, R21, R22, R23, R24, R25, R26: 10, symbol Device:R
Connections:
- new net: DSub2.13, R18.1, R26.2
- new net: DSub2.10, R15.1, R23.2
- new net: DSub2.7, R12.1, R20.2
- new net: DSub2.9, R14.1, R22.2
- new net: DSub2.6, R11.1, R19.2
- new net: DSub2.12, R17.1, R25.2
- new net: DSub2.11, R16.1, R24.2
- new net: DSub2.8, R13.1, R21.2
- new net +24V_AUX: DSub2.23, DSub2.24, DSub2.25
- new net BLNK_AOTF13: R26.1
- new net CH1_AOTF12: R25.1
- new net CH2_AOTF11: R24.1
- new net CH3_AOTF10: R23.1
- new net CH4_AOTF09: R22.1
- new net CH5_AOTF08: R21.1
- new net CH6_AOTF07: R19.1
- new net CH7_AOTF06: R20.1
- new net GND: DSub2.14, DSub2.15, DSub2.16, R11.2, R12.2, R13.2, R14.2, R15.2, R16.2, R17.2, R18.2
- no-connect marks 0 -> 13

Commit message: footprint selection
Parts:
- R11, R12, R13, R14, R15, R16, R17, R18, R19, R20, R21, R22, R23, R24, R25, R26: footprint (none) -> Resistor_SMD:R_0603_1608Metric
Changed lines of the file:
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@@
 			)
 		)
-		(property "Footprint" ""
+		(property "Footprint" "Resistor_SMD:R_0603_1608Metric"
 			(at 163.322 119.38 90)
 			(hide yes)
@@
 			)
 		)
-		(property "Footprint" ""
+		(property "Footprint" "Resistor_SMD:R_0603_1608Metric"
 			(at 97.79 146.558 90)
 			(hide yes)
@@
 			)
 		)
-		(property "Footprint" ""
+		(property "Footprint" "Resistor_SMD:R_0603_1608Metric"
 			(at 148.082 119.38 90)
 			(hide yes)
@@
 			)
 		)
-		(property "Footprint" ""
+		(property "Footprint" "Resistor_SMD:R_0603_1608Metric"
 			(at 132.842 119.38 90)
 			(hide yes)
@@
 			)
 		)
-		(property "Footprint" ""
+		(property "Footprint" "Resistor_SMD:R_0603_1608Metric"
 			(at 97.79 95.758 90)
 			(hide yes)
@@
 			)
 		)
-		(property "Footprint" ""
+		(property "Footprint" "Resistor_SMD:R_0603_1608Metric"
 			(at 127.762 119.38 90)
 			(hide yes)
@@
 			)
 		)
-		(property "Footprint" ""
+		(property "Footprint" "Resistor_SMD:R_0603_1608Metric"
 			(at 158.242 119.38 90)
 			(hide yes)
@@
 			)
 		)
-		(property "Footprint" ""
+		(property "Footprint" "Resistor_SMD:R_0603_1608Metric"
 			(at 153.162 119.38 90)
 			(hide yes)
@@
 			)
 		)
-		(property "Footprint" ""
+		(property "Footprint" "Resistor_SMD:R_0603_1608Metric"
 			(at 97.79 83.058 90)
 			(hide yes)
@@
 			)
 		)
-		(property "Footprint" ""
+		(property "Footprint" "Resistor_SMD:R_0603_1608Metric"
 			(at 97.79 121.158 90)
 			(hide yes)
@@
 			)
 		)
-		(property "Footprint" ""
+		(property "Footprint" "Resistor_SMD:R_0603_1608Metric"
 			(at 97.79 108.458 90)
 			(hide yes)
@@
 			)
 		)
-		(property "Footprint" ""
+		(property "Footprint" "Resistor_SMD:R_0603_1608Metric"
 			(at 143.002 119.38 90)
 			(hide yes)
@@
 			)
 		)
-		(property "Footprint" ""
+		(property "Footprint" "Resistor_SMD:R_0603_1608Metric"
 			(at 97.79 57.658 90)
 			(hide yes)
@@
 			)
 		)
-		(property "Footprint" ""
+		(property "Footprint" "Resistor_SMD:R_0603_1608Metric"
 			(at 137.922 119.38 90)
 			(hide yes)
@@
 			)
 		)
-		(property "Footprint" ""
+		(property "Footprint" "Resistor_SMD:R_0603_1608Metric"
 			(at 97.79 133.858 90)
 			(hide yes)
@@
 			)
 		)
-		(property "Footprint" ""
+		(property "Footprint" "Resistor_SMD:R_0603_1608Metric"
 			(at 97.79 70.358 90)
 			(hide yes)

Commit message: initial layout
Connections:
- net CH6_AOTF07: now also R20.1; no longer R19.1
- net CH7_AOTF06: now also R19.1; no longer R20.1
Changed lines of the file:
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@@
 	(global_label "CH7_AOTF06"
+		(shape input)
+		(at 82.55 55.88 180)
+		(fields_autoplaced yes)
+		(effects
+			(font
+				(size 1.27 1.27)
+			)
+			(justify right)
+		)
+		(property "Intersheetrefs" "${INTERSHEET_REFS}"
+			(at 67.8929 55.88 0)
+			(hide yes)
+			(show_name no)
+			(do_not_autoplace no)
+			(effects
+				(font
+					(size 1.27 1.27)
+				)
+				(justify right)
+			)
+		)
+	)
+	(global_label "CH6_AOTF07"
 		(shape input)
 		(at 82.55 68.58 180)
@@
 			(hide yes)
 			(show_name no)
-			(do_not_autoplace no)
-			(effects
-				(font
-					(size 1.27 1.27)
-				)
-				(justify right)
-			)
-		)
-	)
-	(global_label "CH6_AOTF07"
-		(shape input)
-		(at 82.55 55.88 180)
-		(fields_autoplaced yes)
-		(effects
-			(font
-				(size 1.27 1.27)
-			)
-			(justify right)
-		)
-		(property "Intersheetrefs" "${INTERSHEET_REFS}"
-			(at 67.8929 55.88 0)
-			(hide yes)
-			(show_name no)
