File: Analog_Switch.kicad_sch (KiCad schematic)
At the start: 0 parts

Commit message: schematic complete
Parts:
- added C10, C11, C12, C13: 220n, symbol Device:C
- added C7, C9: 1u, symbol Device:C
- added C8: 22u, symbol Device:C
- added U2: REF5050ID, Package_SO:SOIC-8_3.9x4.9mm_P1.27mm, symbol Reference_Voltage:REF5050ID
- added U3, U4: ADG1634BRUZ-REEL7, Imported:TSSOP-20_L6.5-W4.4-P0.65-LS6.4-BL, symbol Imported:ADG1634BRUZ-REEL7
- added U5, U6: OPA4192IDR, Imported:SOIC-14_L8.7-W3.9-P1.27-LS6.0-BL, symbol Imported:OPA4192IDR
Connections:
- new net: C9.1, U2.5 (Trim/NR)
- new net +5V_REF: C8.1, U2.6 (Vout), U3.12 (S3A), U3.19 (S4A), U3.2 (S1A), U3.9 (S2A), U4.12 (S3A), U4.19 (S4A), U4.2 (S1A), U4.9 (S2A)
- new net +6V: C10.1, C11.1, C12.2, C13.2, C7.1, U2.2 (Vin), U3.16 (VDD), U4.16 (VDD), U5.4 (V+), U6.4 (V+)
- new net BLNK: U3.3 (D1), U5.3 (+INA)
- new net BLNK_AOTF13: U5.1 (OUTA), U5.2 (-INA)
- new net BLNK_NI3_DIO29: U3.1 (IN1)
- new net CH1: U3.8 (D2), U5.5 (+INB)
- new net CH1_AOTF12: U5.6 (-INB), U5.7 (OUTB)
- new net CH1_NI7_DIO25: U3.10 (IN2)
- new net CH2: U3.13 (D3), U5.10 (+INC)
- new net CH2_AOTF11: U5.8 (OUTC), U5.9 (-INC)
- new net CH2_NI11_DIO21: U3.11 (IN3)
- new net CH3: U3.18 (D4), U5.12 (+IND)
- new net CH3_AOTF10: U5.13 (-IND), U5.14 (OUTD)
- new net CH3_NI15_DIO17: U3.20 (IN4)
- new net CH4: U4.3 (D1), U6.3 (+INA)
- new net CH4_AOTF09: U6.1 (OUTA), U6.2 (-INA)
- new net CH4_NI19_DIO13: U4.1 (IN1)
- new net CH5: U4.8 (D2), U6.5 (+INB)
- new net CH5_AOTF08: U6.6 (-INB), U6.7 (OUTB)
- new net CH5_NI23_DIO9: U4.10 (IN2)
- new net CH6: U4.13 (D3), U6.10 (+INC)
- new net CH6_AOTF07: U6.8 (OUTC), U6.9 (-INC)
- new net CH6_NI27_DIO5: U4.11 (IN3)
- new net CH7: U4.18 (D4), U6.12 (+IND)
- new net CH7_AOTF06: U6.13 (-IND), U6.14 (OUTD)
- new net CH7_NI31_DIO1: U4.20 (IN4)
- new net GND: C10.2, C11.2, C12.1, C13.1, C7.2, C8.2, C9.2, U2.4 (GND), U3.14 (S3B), U3.17 (S4B), U3.4 (S1B), U3.5 (VSS), U3.6 (GND), U3.7 (S2B), U4.14 (S3B), U4.17 (S4B), U4.4 (S1B), U4.5 (VSS), U4.6 (GND), U4.7 (S2B), U5.11 (V-), U6.11 (V-)
- no-connect marks 0 -> 3
Other:
- note added: "5V Reference"
- note added: "Global labels look nicer this way"
- note added: "Op Amps"
- note added: "Switch"

Commit message: footprint selection
Parts:
- C10, C11, C12, C13: footprint (none) -> Capacitor_SMD:C_0805_2012Metric
- C7, C9: footprint (none) -> Capacitor_SMD:C_0603_1608Metric
- C8: footprint (none) -> Capacitor_SMD:C_1206_3216Metric
Changed lines of the file:
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@@
 			)
 		)
-		(property "Footprint" ""
+		(property "Footprint" "Capacitor_SMD:C_0603_1608Metric"
 			(at 59.9948 67.31 0)
 			(hide yes)
@@
 			)
 		)
-		(property "Footprint" ""
+		(property "Footprint" "Capacitor_SMD:C_0603_1608Metric"
 			(at 35.8648 45.72 0)
 			(hide yes)
@@
 			)
 		)
-		(property "Footprint" ""
+		(property "Footprint" "Capacitor_SMD:C_1206_3216Metric"
 			(at 70.8152 62.23 0)
 			(hide yes)
@@
 			)
 		)
-		(property "Footprint" ""
+		(property "Footprint" "Capacitor_SMD:C_0805_2012Metric"
 			(at 201.93 124.7648 0)
 			(hide yes)
@@
 			)
 		)
-		(property "Footprint" ""
+		(property "Footprint" "Capacitor_SMD:C_0805_2012Metric"
 			(at 120.65 124.7648 0)
 			(hide yes)
@@
 			)
 		)
-		(property "Footprint" ""
+		(property "Footprint" "Capacitor_SMD:C_0805_2012Metric"
 			(at 245.11 54.9148 0)
 			(hide yes)
@@
 			)
 		)
-		(property "Footprint" ""
+		(property "Footprint" "Capacitor_SMD:C_0805_2012Metric"
 			(at 162.56 56.1848 0)
 			(hide yes)

Commit message: initial layout
Connections:
- net BLNK: now also U4.18 (D4), U6.3 (+INA); no longer U3.3 (D1), U5.3 (+INA)
- net BLNK_AOTF13: now also U6.1 (OUTA), U6.2 (-INA); no longer U5.1 (OUTA), U5.2 (-INA)
- net BLNK_NI3_DIO29: now also U4.20 (IN4); no longer U3.1 (IN1)
- net CH1: now also U4.13 (D3), U6.5 (+INB); no longer U3.8 (D2), U5.5 (+INB)
- net CH1_AOTF12: now also U6.6 (-INB), U6.7 (OUTB); no longer U5.6 (-INB), U5.7 (OUTB)
- net CH1_NI7_DIO25: now also U4.11 (IN3); no longer U3.10 (IN2)
- net CH2: now also U4.8 (D2), U6.10 (+INC); no longer U3.13 (D3), U5.10 (+INC)
- net CH2_AOTF11: now also U6.8 (OUTC), U6.9 (-INC); no longer U5.8 (OUTC), U5.9 (-INC)
- net CH2_NI11_DIO21: now also U4.10 (IN2); no longer U3.11 (IN3)
- net CH3: now also U4.3 (D1), U6.12 (+IND); no longer U3.18 (D4), U5.12 (+IND)
- net CH3_AOTF10: now also U6.13 (-IND), U6.14 (OUTD); no longer U5.13 (-IND), U5.14 (OUTD)
- net CH3_NI15_DIO17: now also U4.1 (IN1); no longer U3.20 (IN4)
- net CH4: now also U3.18 (D4), U5.3 (+INA); no longer U4.3 (D1), U6.3 (+INA)
- net CH4_AOTF09: now also U5.1 (OUTA), U5.2 (-INA); no longer U6.1 (OUTA), U6.2 (-INA)
- net CH4_NI19_DIO13: now also U3.20 (IN4); no longer U4.1 (IN1)
- net CH5: now also U3.13 (D3), U5.5 (+INB); no longer U4.8 (D2), U6.5 (+INB)
- net CH5_AOTF08: now also U5.6 (-INB), U5.7 (OUTB); no longer U6.6 (-INB), U6.7 (OUTB)
- net CH5_NI23_DIO9: now also U3.11 (IN3); no longer U4.10 (IN2)
- net CH6: now also U3.8 (D2), U5.10 (+INC); no longer U4.13 (D3), U6.10 (+INC)
- net CH6_AOTF07: now also U5.8 (OUTC), U5.9 (-INC); no longer U6.8 (OUTC), U6.9 (-INC)
- net CH6_NI27_DIO5: now also U3.10 (IN2); no longer U4.11 (IN3)
- net CH7: now also U3.3 (D1), U5.12 (+IND); no longer U4.18 (D4), U6.12 (+IND)
- net CH7_AOTF06: now also U5.13 (-IND), U5.14 (OUTD); no longer U6.13 (-IND), U6.14 (OUTD)
- net CH7_NI31_DIO1: now also U3.1 (IN1); no longer U4.20 (IN4)
Other:
- moved on the sheet: U3, U4, U5, U6
