File: FPGA_Input.kicad_sch (KiCad schematic)
At the start: 0 parts

Commit message: fpga connector
Parts:
- added DSUB1: 2-5174225-5, Imported:DSUB-TH_68P_2-5174225-5, symbol Imported:2-5174225-5
- added R10, R3, R4, R5, R6, R7, R8, R9: 10k, symbol Device:R_Small
Connections:
- new net BLNK_NI3_DIO29: DSUB1.A3, R3.1
- new net CH1_NI7_DIO25: DSUB1.A7, R4.1
- new net CH2_NI11_DIO21: DSUB1.A11, R5.1
- new net CH3_NI15_DIO17: DSUB1.A15, R6.1
- new net CH4_NI19_DIO13: DSUB1.A19, R7.1
- new net CH5_NI23_DIO9: DSUB1.A23, R8.1
- new net CH6_NI27_DIO5: DSUB1.A27, R9.1
- new net CH7_NI31_DIO1: DSUB1.A31, R10.1
- new net GND: DSUB1.A10, DSUB1.A12, DSUB1.A14, DSUB1.A16, DSUB1.A18, DSUB1.A2, DSUB1.A20, DSUB1.A22, DSUB1.A24, DSUB1.A26, DSUB1.A28, DSUB1.A30, DSUB1.A32, DSUB1.A33, DSUB1.A34, DSUB1.A4, DSUB1.A6, DSUB1.A8, DSUB1.B10, DSUB1.B12, DSUB1.B14, DSUB1.B16, DSUB1.B18, DSUB1.B2, DSUB1.B20, DSUB1.B22, DSUB1.B24, DSUB1.B26, DSUB1.B28, DSUB1.B30, DSUB1.B32, DSUB1.B33, DSUB1.B34, DSUB1.B4, DSUB1.B6, DSUB1.B8, R10.2, R3.2, R4.2, R5.2, R6.2, R7.2, R8.2, R9.2
- no-connect marks 0 -> 24
Other:
- note added: "Pull down resistors provide a defined off state"

Commit message: footprint selection
Parts:
- R10, R3, R4, R5, R6, R7, R8, R9: footprint (none) -> Resistor_SMD:R_0603_1608Metric
Changed lines of the file:
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@@
 			)
 		)
-		(property "Footprint" ""
+		(property "Footprint" "Resistor_SMD:R_0603_1608Metric"
 			(at 114.3 80.01 0)
 			(hide yes)
@@
 			)
 		)
-		(property "Footprint" ""
+		(property "Footprint" "Resistor_SMD:R_0603_1608Metric"
 			(at 114.3 130.81 0)
 			(hide yes)
@@
 			)
 		)
-		(property "Footprint" ""
+		(property "Footprint" "Resistor_SMD:R_0603_1608Metric"
 			(at 114.3 59.69 0)
 			(hide yes)
@@
 			)
 		)
-		(property "Footprint" ""
+		(property "Footprint" "Resistor_SMD:R_0603_1608Metric"
 			(at 114.3 100.33 0)
 			(hide yes)
@@
 			)
 		)
-		(property "Footprint" ""
+		(property "Footprint" "Resistor_SMD:R_0603_1608Metric"
 			(at 114.3 110.49 0)
 			(hide yes)
@@
 			)
 		)
-		(property "Footprint" ""
+		(property "Footprint" "Resistor_SMD:R_0603_1608Metric"
 			(at 114.3 120.65 0)
 			(hide yes)
@@
 			)
 		)
-		(property "Footprint" ""
+		(property "Footprint" "Resistor_SMD:R_0603_1608Metric"
 			(at 114.3 69.85 0)
 			(hide yes)
@@
 			)
 		)
-		(property "Footprint" ""
+		(property "Footprint" "Resistor_SMD:R_0603_1608Metric"
 			(at 114.3 90.17 0)
 			(hide yes)

Commit message: initial layout
Connections:
- net BLNK_NI3_DIO29: now also DSUB1.A31, R10.1; no longer DSUB1.A3, R3.1
- net CH1_NI7_DIO25: now also DSUB1.A27, R9.1; no longer DSUB1.A7, R4.1
- net CH2_NI11_DIO21: now also DSUB1.A23, R8.1; no longer DSUB1.A11, R5.1
- net CH3_NI15_DIO17: now also DSUB1.A19, R7.1; no longer DSUB1.A15, R6.1
- net CH4_NI19_DIO13: now also DSUB1.A15, R6.1; no longer DSUB1.A19, R7.1
- net CH5_NI23_DIO9: now also DSUB1.A11, R5.1; no longer DSUB1.A23, R8.1
- net CH6_NI27_DIO5: now also DSUB1.A7, R4.1; no longer DSUB1.A27, R9.1
- net CH7_NI31_DIO1: now also DSUB1.A3, R3.1; no longer DSUB1.A31, R10.1
Changed lines of the file:
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@@
 	(global_label "CH3_NI15_DIO17"
+		(shape input)
+		(at 88.9 96.52 180)
+		(fields_autoplaced yes)
+		(effects
+			(font
+				(size 1.27 1.27)
+			)
+			(justify right)
+		)
+		(property "Intersheetrefs" "${INTERSHEET_REFS}"
+			(at 70.191 96.52 0)
+			(hide yes)
+			(show_name no)
+			(do_not_autoplace no)
+			(effects
+				(font
+					(size 1.27 1.27)
+				)
+				(justify right)
+			)
+		)
+	)
+	(global_label "CH4_NI19_DIO13"
 		(shape input)
 		(at 88.9 86.36 180)
@@
 		)
 	)
-	(global_label "CH4_NI19_DIO13"
+	(global_label "CH6_NI27_DIO5"
 		(shape input)
-		(at 88.9 96.52 180)
+		(at 88.9 66.04 180)
 		(fields_autoplaced yes)
 		(effects
@@
 		)
 		(property "Intersheetrefs" "${INTERSHEET_REFS}"
-			(at 70.191 96.52 0)
+			(at 71.4005 66.04 0)
 			(hide yes)
 			(show_name no)
@@
 		)
 	)
-	(global_label "CH6_NI27_DIO5"
+	(global_label "CH7_NI31_DIO1"
+		(shape input)
+		(at 88.9 55.88 180)
+		(fields_autoplaced yes)
+		(effects
+			(font
+				(size 1.27 1.27)
+			)
+			(justify right)
+		)
+		(property "Intersheetrefs" "${INTERSHEET_REFS}"
+			(at 71.4005 55.88 0)
+			(hide yes)
+			(show_name no)
+			(do_not_autoplace no)
+			(effects
+				(font
+					(size 1.27 1.27)
+				)
+				(justify right)
+			)
+		)
+	)
+	(global_label "CH5_NI23_DIO9"
+		(shape input)
+		(at 88.9 76.2 180)
+		(fields_autoplaced yes)
+		(effects
+			(font
+				(size 1.27 1.27)
+			)
+			(justify right)
+		)
+		(property "Intersheetrefs" "${INTERSHEET_REFS}"
+			(at 71.4005 76.2 0)
+			(hide yes)
+			(show_name no)
+			(do_not_autoplace no)
+			(effects
+				(font
+					(size 1.27 1.27)
+				)
+				(justify right)
+			)
+		)
+	)
+	(global_label "BLNK_NI3_DIO29"
+		(shape input)
+		(at 88.9 127 180)
+		(fields_autoplaced yes)
+		(effects
+			(font
+				(size 1.27 1.27)
+			)
+			(justify right)
+		)
+		(property "Intersheetrefs" "${INTERSHEET_REFS}"
+			(at 70.3119 127 0)
+			(hide yes)
+			(show_name no)
+			(do_not_autoplace no)
+			(effects
+				(font
+					(size 1.27 1.27)
+				)
+				(justify right)
+			)
+		)
+	)
+	(global_label "CH1_NI7_DIO25"
 		(shape input)
 		(at 88.9 116.84 180)
@@
 		)
 	)
-	(global_label "CH7_NI31_DIO1"
-		(shape input)
-		(at 88.9 127 180)
-		(fields_autoplaced yes)
-		(effects
-			(font
-				(size 1.27 1.27)
-			)
-			(justify right)
-		)
-		(property "Intersheetrefs" "${INTERSHEET_REFS}"
-			(at 71.4005 127 0)
-			(hide yes)
-			(show_name no)
-			(do_not_autoplace no)
-			(effects
-				(font
-					(size 1.27 1.27)
-				)
-				(justify right)
-			)
-		)
-	)
-	(global_label "CH5_NI23_DIO9"
+	(global_label "CH2_NI11_DIO21"
 		(shape input)
 		(at 88.9 106.68 180)
@@
 		)
 		(property "Intersheetrefs" "${INTERSHEET_REFS}"
-			(at 71.4005 106.68 0)
+			(at 70.191 106.68 0)
 			(hide yes)
 			(show_name no)
-			(do_not_autoplace no)
-			(effects
-				(font
-					(size 1.27 1.27)
-				)
-				(justify right)
-			)
-		)
-	)
-	(global_label "BLNK_NI3_DIO29"
-		(shape input)
-		(at 88.9 55.88 180)
-		(fields_autoplaced yes)
-		(effects
-			(font
-				(size 1.27 1.27)
-			)
-			(justify right)
-		)
-		(property "Intersheetrefs" "${INTERSHEET_REFS}"
-			(at 70.3119 55.88 0)
-			(hide yes)
-			(show_name no)
-			(do_not_autoplace no)
-			(effects
-				(font
-					(size 1.27 1.27)
-				)
-				(justify right)
-			)
-		)
-	)
-	(global_label "CH1_NI7_DIO25"
-		(shape input)
-		(at 88.9 66.04 180)
-		(fields_autoplaced yes)
-		(effects
-			(font
-				(size 1.27 1.27)
-			)
-			(justify right)
-		)
-		(property "Intersheetrefs" "${INTERSHEET_REFS}"
-			(at 71.4005 66.04 0)
-			(hide yes)
-			(show_name no)
-			(do_not_autoplace no)
-			(effects
-				(font
-					(size 1.27 1.27)
-				)
-				(justify right)
-			)
-		)
-	)
-	(global_label "CH2_NI11_DIO21"
-		(shape input)
-		(at 88.9 76.2 180)
-		(fields_autoplaced yes)
-		(effects
-			(font
-				(size 1.27 1.27)
-			)
-			(justify right)
-		)
-		(property "Intersheetrefs" "${INTERSHEET_REFS}"
-			(at 70.191 76.2 0)
-			(hide yes)
-			(show_name no)
