File: iAOLLS_AOTF_FPGA_Interface.kicad_pcb (KiCad board)
At the start: 2 copper layers, 6.5 x 63.9 mm, 50 parts, among them U1 LMR36510ADDA, U2 REF5050ID, U3 ADG1634BRUZ-REEL7, U4 ADG1634BRUZ-REEL7, U5 OPA4192IDR, U6 OPA4192IDR

Commit message: reset layout
Parts:
- moved C9 33.2 mm to (154.8, 68.0), turned to 0 degrees
- moved C7 31.1 mm to (152.3, 78.2), turned to 0 degrees
- moved R22 29.8 mm to (125.7, 88.4), turned to -90 degrees
- moved R19 29.8 mm to (125.7, 76.5), turned to 90 degrees
- moved R26 28.9 mm to (126.2, 108.0), turned to -90 degrees
- moved U2 28.6 mm to (151.6, 73.2), turned to 90 degrees
- moved R23 28.6 mm to (126.2, 96.3), turned to 90 degrees
- moved R11 27.2 mm to (154.4, 90.6)
- moved C8 26.1 mm to (149.7, 68.0), turned to 180 degrees
- moved C13 25.4 mm to (130.6, 87.6), turned to 180 degrees
- moved R12 25.0 mm to (154.4, 94.1)
- moved R13 23.6 mm to (154.4, 97.7)
- moved R14 22.2 mm to (154.4, 101.3)
- moved C12 19.2 mm to (131.1, 107.2), turned to 180 degrees
- moved R15 19.2 mm to (154.4, 104.8)
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Routing:
- net CH7_NI31_DIO1: track 3.98 -> 0.00 mm
- net CH6_NI27_DIO5: track 3.98 -> 0.00 mm
- net CH5_NI23_DIO9: track 3.97 -> 0.00 mm
- net CH4_NI19_DIO13: track 3.97 -> 0.00 mm
- net CH3_NI15_DIO17: track 3.96 -> 0.00 mm
- net CH2_NI11_DIO21: track 3.96 -> 0.00 mm
- net CH1_NI7_DIO25: track 3.96 -> 0.00 mm
- net BLNK_NI3_DIO29: track 3.95 -> 0.00 mm
- net +6V: track 2.93 -> 0.00 mm, vias 0 -> 4
- net GND: track 2.86 -> 0.00 mm

Commit message: edge cut
Parts:
- moved C7 18.5 mm to (133.9, 76.2)
- moved C8 18.5 mm to (131.3, 66.0)
- moved C9 18.5 mm to (136.4, 66.0)
- moved U2 18.5 mm to (133.2, 71.2)
- moved DSub2 14.9 mm to (152.0, 88.0)
- moved R11 12.7 mm to (144.5, 82.7)
- moved R12 12.7 mm to (144.5, 86.3)
- moved R13 12.7 mm to (144.5, 89.8)
- moved R16 12.7 mm to (144.5, 100.5)
- moved R17 12.7 mm to (144.5, 104.1)
- moved R18 12.7 mm to (144.5, 107.6)
- moved R14 12.7 mm to (144.5, 93.4)
- moved R15 12.7 mm to (144.5, 97.0)
- moved C11 2.29 mm to (119.4, 89.7)
- moved C13 2.29 mm to (130.6, 89.9)
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Routing:
- net +6V: vias 4 -> 0
Other:
- board size 6.5 x 63.9 mm -> 66.8 x 77.2 mm

Commit message: complete layout first pass
Parts:
- moved C7 3.19 mm to (130.7, 75.9)
- moved C8 3.18 mm to (128.1, 66.0)
- moved U2 3.18 mm to (130.0, 71.1)
- moved C9 3.18 mm to (133.2, 66.0)
- moved C3 3.14 mm to (130.0, 119.1)
- moved C4 3.14 mm to (130.8, 121.4)
- moved R23 2.75 mm to (128.5, 97.8)
- moved U6 2.62 mm to (132.3, 103.4)
- moved R19 2.62 mm to (128.0, 80.0)
- moved L1 2.59 mm to (127.8, 126.5)
- moved R26 2.50 mm to (128.5, 109.0)
- moved U5 2.41 mm to (131.8, 85.6)
- moved C12 2.40 mm to (132.3, 109.2), turned to 90 degrees
- moved R22 2.34 mm to (128.0, 91.2)
- moved C5 2.30 mm to (120.2, 116.3)
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Routing:
- net GND: track 0.00 -> 121.8 mm, vias 0 -> 211
- net +6V: track 0.00 -> 116.6 mm, vias 0 -> 12
- net +5V_REF: track 0.00 -> 87.7 mm, vias 0 -> 4
- net Net-(DSub2-Pad13): track 0.00 -> 28.9 mm
- net +24V_AUX: track 0.00 -> 26.5 mm
- net Net-(DSub2-Pad6): track 0.00 -> 25.1 mm
- net Net-(DSub2-Pad9): track 0.00 -> 23.6 mm
- net Net-(DSub2-Pad10): track 0.00 -> 22.8 mm
- net BLNK_NI3_DIO29: track 0.00 -> 21.0 mm
- net CH4_NI19_DIO13: track 0.00 -> 19.7 mm
- net CH3_NI15_DIO17: track 0.00 -> 19.5 mm
- net CH7_NI31_DIO1: track 0.00 -> 19.2 mm
- net /Analog Switch/CH2: track 0.00 -> 18.2 mm
- net /Analog Switch/CH5: track 0.00 -> 18.1 mm
- net /Analog Switch/CH6: track 0.00 -> 18.1 mm
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- added copper zone on B.Cu, net GND
- added copper zone on F.Cu, net GND

Commit message: fixing all DRC errors
Routing:
- net GND: track 121.8 -> 33.3 mm, vias 211 -> 210
- net CH5_AOTF08: track 1.27 -> 3.02 mm
- net CH3_AOTF10: track 2.14 -> 3.41 mm
Other:
- board size 66.8 x 77.2 mm -> 66.3 x 77.2 mm

Commit message: fix drc errors and add mounting holes
Parts:
- added H1: MountingHole, MountingHole:MountingHole_3.2mm_M3_Pad_Via, F.Cu at (107.0, 55.0)
- added H2: MountingHole, MountingHole:MountingHole_3.2mm_M3_Pad_Via, F.Cu at (152.0, 55.0)
- added H3: MountingHole, MountingHole:MountingHole_3.2mm_M3_Pad_Via, F.Cu at (107.0, 135.0)
- added H4: MountingHole, MountingHole:MountingHole_3.2mm_M3_Pad_Via, F.Cu at (152.0, 135.0)
Routing:
- net GND: vias 210 -> 244
Other:
- board size 66.3 x 77.2 mm -> 63.4 x 93.3 mm
